Commit message: My modifications for the Dobot package

File: dobot_rviz/urdf/cr5_robot.urdf (robot description, URDF)
Before this commit: robot cr5_robot, 8 links, 7 joints
Links:
- added link zed, mass 0.2; collision box size=0.12 0.10 0.05; visual box size=0.12 0.12 0.05
Joints:
- added joint zed: type fixed, parent Link6, child zed, origin xyz=0 0 0 rpy=0 0 0
